File: Custom PCB esp32c6/esp32c6_daikin.kicad_pcb (KiCad board)
At the start: 2 copper layers, 26 x 43.5 mm, 34 parts, among them J1 1x5, J2 USB_C_Receptacle_USB2.0_16P, Q1 BSS138PS, U1 TPS562246, U2 ESP32-C6-MINI-1/U

Commit message: Add files via upload
Parts:
- removed BootSwitch1, MatterSwitch1, ResetSwitch1: Tactile Button, 160gf, JLCPCB:SW_TS-1088-AR02016
- removed J1: 1x5, EasyEDA2kiCad:CONN-TH_S5B-EH-LF-SN
- removed R4, R7: 5.1k, EasyEDA2kiCad:R0402
- added Boot1: Tactile Button, 160gf, easyeda2kicad:SW-SMD_L3.9-W3.0-P4.45, F.Cu at (160.1, 105.2)
- added Matter1: Tactile Button, 160gf, easyeda2kicad:SW-SMD_L3.9-W3.0-P4.45, F.Cu at (165.2, 107.3)
- added Reset1: Tactile Button, 160gf, easyeda2kicad:SW-SMD_L3.9-W3.0-P4.45, F.Cu at (156.6, 100.5)
- C1, C16, C18, C19, C2, C3, C4, C5, C7, C8: footprint EasyEDA2kiCad:C0402 -> easyeda2kicad:C0402
- C15, C17: footprint EasyEDA2kiCad:C0805 -> easyeda2kicad:C0805
- C6: footprint EasyEDA2kiCad:C0603 -> easyeda2kicad:C0603
- D2, D3: footprint EasyEDA2kiCad:DFN1006-2L_L1.0-W0.6-P0.65-BI -> easyeda2kicad:DFN1006-2L_L1.0-W0.6-P0.65-BI
- D4: footprint EasyEDA2kiCad:D0402 -> easyeda2kicad:D0402
- J2: value USB_C_Receptacle_USB2.0_16P -> Conn_01x07; footprint Connector_USB:USB_C_Receptacle_GCT_USB4105-xx-A_16P_TopMnt_Horizontal -> Connector_PinHeader_2.54mm:PinHeader_1x07_P2.54mm_Horizontal
- L1: footprint EasyEDA2kiCad:IND-SMD_L4.9-W4.9_NRS50XX -> easyeda2kicad:IND-SMD_L4.9-W4.9_NRS50XX
- Q1: footprint EasyEDA2kiCad:SOT-363_L2.0-W1.3-P0.65-LS2.1-BR -> easyeda2kicad:SOT-363_L2.0-W1.3-P0.65-LS2.1-BR
- R1, R2, R8, R9: footprint EasyEDA2kiCad:R0402 -> easyeda2kicad:R0402
- R3: value 10K -> 10k; footprint EasyEDA2kiCad:R0402 -> easyeda2kicad:R0402
- R5, R6: footprint EasyEDA2kiCad:R0603 -> easyeda2kicad:R0603
- U1: footprint EasyEDA2kiCad:SOT-5X3-6_L1.6-W1.2-P0.50-LS1.6-BR -> easyeda2kicad:SOT-5X3-6_L1.6-W1.2-P0.50-LS1.6-BR
- U2: value ESP32-C6-MINI-1/U -> WT0132C6-S5; footprint Espressif:ESP32-C6-MINI-1 -> easyeda2kicad:WT0132C6-S5; moved to B.Cu
- moved J2 114.7 mm to (175.6, 92.0), turned to 0 degrees
- moved D4 113.3 mm to (172.8, 99.9)
- moved D3 112.8 mm to (172.7, 104.2)
- moved R2 111.8 mm to (170.8, 99.9), turned to 0 degrees
- moved R1 111.2 mm to (173.5, 101.5), turned to 90 degrees
- moved Q1 108.6 mm to (170.0, 102.0), turned to 0 degrees
- moved D2 108.3 mm to (170.4, 103.6)
- moved C17 101.8 mm to (173.1, 93.3), turned to 90 degrees
- moved C19 99.9 mm to (169.9, 97.8), turned to -90 degrees
- moved R5 99.6 mm to (171.5, 96.2), turned to 90 degrees
- moved C8 98.9 mm to (157.7, 96.2)
- moved R9 98.9 mm to (158.2, 94.2)
- moved R3 98.8 mm to (159.9, 94.7), turned to 90 degrees
- moved R8 98.7 mm to (172.5, 98.4), turned to 0 degrees
- moved R6 97.7 mm to (167.7, 98.2)
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Connections:
- C1 pad 2: /3.3V -> 3V3
- C15 pad 1: /3.3V -> 3V3
- C16 pad 1: /12V -> V_in
- C17 pad 1: /12V -> V_in
- C19 pad 2: /3.3V -> 3V3
- C2 pad 2: /3.3V -> 3V3
- C3 pad 1: /12V -> V_in
- C4 pad 2: /3.3V -> 3V3
- C5 pad 2: /3.3V -> 3V3
- C6 pad 1: Net-(U2-EN/CHIP_PU) -> Net-(U2-EN)
- C7 pad 2: /3.3V -> 3V3
- D2 pad 2: /Pin 3 -> Net-(J2-Pin_3)
- L1 pad 2: /3.3V -> 3V3
- Q1 pad 3: /Pin 3 -> Net-(J2-Pin_3)
- Q1 pad 5: /TX -> TX1
- Q1 pad 6: /RX -> RX1
- R1 pad 1: Net-(J1-Pin_5) -> Net-(J2-Pin_5)
- R1 pad 2: /Pin 3 -> Net-(J2-Pin_3)
- R2 pad 1: /3.3V -> 3V3
- R3 pad 1: /3.3V -> 3V3
- R3 pad 2: Net-(U2-EN/CHIP_PU) -> Net-(U2-EN)
- R5 pad 2: /12V -> V_in
- R6 pad 1: /3.3V -> 3V3
- R9 pad 2: Net-(U2-EN/CHIP_PU) -> Net-(U2-EN)
- U1 pad 1: /12V -> V_in
- U2 pad 1: GND -> unconnected-(U2-GPIO0-Pad1)
- U2 pad 11: GND -> unconnected-(U2-GPIO8-Pad11)
- U2 pad 12: unconnected-(U2-GPIO0/ADC1_CH0/XTAL_32K_P-Pad12) -> Net-(Boot1-A)
- U2 pad 14: GND -> unconnected-(U2-GPIO3-Pad14)
- U2 pad 15: unconnected-(U2-MTCK/GPIO6/ADC1_CH6-Pad15) -> RX0
- U2 pad 16: unconnected-(U2-MTDO/GPIO7-Pad16) -> TX0
- U2 pad 17: Net-(U2-GPIO12/USB_D-) -> unconnected-(U2-GPIO18-Pad17)
- U2 pad 18: Net-(U2-GPIO13/USB_D+) -> unconnected-(U2-GPIO19-Pad18)
- U2 pad 19: unconnected-(U2-GPIO14-Pad19) -> RX1
- U2 pad 2: GND -> unconnected-(U2-GPIO1-Pad2)
- U2 pad 20: unconnected-(U2-GPIO15-Pad20) -> TX1
- U2 pad 22: unconnected-(U2-GPIO8-Pad22) -> Net-(Matter1-A)
- U2 pad 3: /3.3V -> Net-(U2-EN)
- U2 pad 8: Net-(U2-EN/CHIP_PU) -> 3V3
- U2 pad 9: unconnected-(U2-MTMS/GPIO4/ADC1_CH4-Pad9) -> GND
Routing:
- net /3.3V: track 75.1 -> 0.00 mm, vias 4 -> 0
- net /12V: track 59.5 -> 0.00 mm, vias 3 -> 0
- net 3V3: track 0.00 -> 53.7 mm, vias 0 -> 1
- net /RX: track 34.7 -> 0.00 mm, vias 2 -> 0
- net /TX: track 30.2 -> 0.00 mm, vias 2 -> 0
- net TX0: track 0.00 -> 21.6 mm, vias 0 -> 1
- net Net-(U2-GPIO13/USB_D+): track 21.6 -> 0.00 mm, vias 2 -> 0
- net /Pin 3: track 21.1 -> 0.00 mm
- net RX0: track 0.00 -> 19.6 mm, vias 0 -> 1
- net Net-(BootSwitch1-A): track 16.0 -> 0.00 mm, vias 2 -> 0
- net Net-(U2-GPIO12/USB_D-): track 15.9 -> 0.00 mm
- net Net-(J2-Pin_3): track 0.00 -> 13.6 mm
- net V_in: track 0.00 -> 12.2 mm
- net Net-(U2-EN): track 0.00 -> 9.60 mm, vias 0 -> 1
- net Net-(Matter1-A): track 0.00 -> 7.88 mm, vias 0 -> 1
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Other:
- board size 26 x 43.5 mm -> 31.6 x 19.8 mm
- board text added: "RX0"
- board text added: "RX1"
- board text added: "TX0"
- board text added: "TX1"
- board text added: "V_in"
- board text removed: "12V"
- board text removed: "Daikin s21 ESP-C6 v1"
- board text removed: "RX"
- board text removed: "TX"
