File: Custom PCB esp32c6/esp32c6_daikin.kicad_sch (KiCad schematic)
At the start: 34 parts, among them J1 1x5, J2 USB_C_Receptacle_USB2.0_16P, Q1 BSS138PS, U1 TPS562246, U2 ESP32-C6-MINI-1/U

Commit message: Add files via upload
Parts:
- removed J1: 1x5, EasyEDA2kiCad:CONN-TH_S5B-EH-LF-SN, symbol Connector_Generic:Conn_01x05
- removed J2: USB_C_Receptacle_USB2.0_16P, Connector_USB:USB_C_Receptacle_GCT_USB4105-xx-A_16P_TopMnt_Horizontal, symbol Connector:USB_C_Receptacle_USB2.0_16P
- removed R4, R7: 5.1k, EasyEDA2kiCad:R0402, symbol Device:R
- removed U2: ESP32-C6-MINI-1/U, Espressif:ESP32-C6-MINI-1, symbol Espressif:ESP32-C6-MINI-1/U
- added J2: Conn_01x07, Connector_PinHeader_2.54mm:PinHeader_1x07_P2.54mm_Horizontal, symbol Connector_Generic:Conn_01x07
- added U2: WT0132C6-S5, easyeda2kicad:WT0132C6-S5, symbol easyeda2kicad:WT0132C6-S5
- Boot1: renamed from BootSwitch1; footprint JLCPCB:SW_TS-1088-AR02016 -> easyeda2kicad:SW-SMD_L3.9-W3.0-P4.45
- C1, C16, C18, C19, C2, C3, C4, C5, C7, C8: footprint EasyEDA2kiCad:C0402 -> easyeda2kicad:C0402
- C15, C17: footprint EasyEDA2kiCad:C0805 -> easyeda2kicad:C0805
- C6: footprint EasyEDA2kiCad:C0603 -> easyeda2kicad:C0603
- D2, D3: value ~ -> (none); footprint EasyEDA2kiCad:DFN1006-2L_L1.0-W0.6-P0.65-BI -> easyeda2kicad:DFN1006-2L_L1.0-W0.6-P0.65-BI
- D4: footprint EasyEDA2kiCad:D0402 -> easyeda2kicad:D0402
- L1: footprint EasyEDA2kiCad:IND-SMD_L4.9-W4.9_NRS50XX -> easyeda2kicad:IND-SMD_L4.9-W4.9_NRS50XX
- Matter1: renamed from MatterSwitch1; footprint JLCPCB:SW_TS-1088-AR02016 -> easyeda2kicad:SW-SMD_L3.9-W3.0-P4.45
- Q1: footprint EasyEDA2kiCad:SOT-363_L2.0-W1.3-P0.65-LS2.1-BR -> easyeda2kicad:SOT-363_L2.0-W1.3-P0.65-LS2.1-BR
- R1, R2, R8, R9: footprint EasyEDA2kiCad:R0402 -> easyeda2kicad:R0402
- R3: value 10K -> 10k; footprint EasyEDA2kiCad:R0402 -> easyeda2kicad:R0402
- R5, R6: footprint EasyEDA2kiCad:R0603 -> easyeda2kicad:R0603
- Reset1: renamed from ResetSwitch1; footprint JLCPCB:SW_TS-1088-AR02016 -> easyeda2kicad:SW-SMD_L3.9-W3.0-P4.45
- U1: footprint EasyEDA2kiCad:SOT-5X3-6_L1.6-W1.2-P0.50-LS1.6-BR -> easyeda2kicad:SOT-5X3-6_L1.6-W1.2-P0.50-LS1.6-BR
Connections:
- net GND: now also J2.1 (Pin_1), U2.9 (GND)
- net at D3.2, D4.1 (K), Q1.2 (GN): now also J2.4 (Pin_4)
- net at C6.1, R3.2, R9.2: now also U2.3 (EN)
- net at R1.1: now also J2.5 (Pin_5)
- net at Matter1.1 (A): now also U2.22 (GPIO23)
- net at Boot1.1 (A): now also U2.12 (GPIO9)
- net 12V renamed V_in
- net V_in: now also J2.2 (Pin_2)
- net 3.3V renamed 3V3
- net 3V3: now also U2.8 (3V3)
- net Pin 3: no longer names the net of D2.2, Q1.3 (SP), R1.2
- net Pin 3: now also J2.3 (Pin_3)
- net RX renamed RX1
- net RX1: now also U2.19 (GPIO20)
- net TX renamed TX1
- net TX1: now also U2.20 (GPIO21)
- new net RX0: J2.7 (Pin_7), U2.15 (RXD)
- new net TX0: J2.6 (Pin_6), U2.16 (TXD)
- no-connect marks 18 -> 0
Other:
- title: Daikin ESP32-C6-MINI-1 -> Daikin  WT0132C6-S5
- moved on the sheet: Boot1, C6, C8, D2, D3, D4, Matter1, Q1A, Q1B, R2, R3, R9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
